Commit message: feat Converted the camera to a RGB-Depth camera
Converted the robot's camera to be like a Kinect.
It uses the libgazebo_ros_openni_kinect.so library instead.
It generates a point cloud as well as images

File: my_robot/urdf/my_robot.xacro (robot description, xacro)
@@ -14,4 +14,9 @@
     <axis xyz="0 1 0"/>
   </joint>
+  <joint name="camera_optical_joint" type="fixed">
+    <origin xyz="0 0 0" rpy="-1.5707 0 -1.5707"/>
+    <parent link="camera"/>
+    <child link="camera_link_optical"/>
+  </joint>
   <joint name="hokuyo_joint" type="fixed">
     <origin xyz="0.15 0 0.32" rpy="0 0 0"/>
@@ -330,4 +335,6 @@
     </collision>
   </link>
+  <link name="camera_link_optical">
+  </link>
   <link name='hokuyo'>
     <pose>0 0 0 0 0 0</pose>
